File: weather_station_dc/weather_station_dc/weather_station_dc.sch (KiCad schematic (older format))
At the start: 17 parts

Commit message: updates for ws
Parts:
- added D1: D, symbol Device:D
- gave numbers to parts that had none: 17
Connections:
- net +12V: now also D1.1 (K)
- net at J6.2 (Pin_2), Q1.2 (C): now also D1.2 (A)
Changed lines of the file:
@@
 $EndDescr
 $Comp
-L Arduino_MYS:ArduinoProMini IC?
+L Arduino_MYS:ArduinoProMini IC1
 U 1 1 5FAD02F7
 P 4600 4650
-F 0 "IC?" H 4650 6100 40  0000 C CNN
+F 0 "IC1" H 4650 6100 40  0000 C CNN
 F 1 "ArduinoProMini" H 4650 6024 40  0000 C CNN
 F 2 "mysensors_arduino:pro_mini_china" H 4600 4650 30  0001 C CIN
@@
 $EndComp
 $Comp
-L Transistor_BJT:TIP120 Q?
+L Transistor_BJT:TIP120 Q1
 U 1 1 5FAD55AF
 P 8350 5900
-F 0 "Q?" H 8557 5946 50  0000 L CNN
+F 0 "Q1" H 8557 5946 50  0000 L CNN
 F 1 "TIP120" H 8557 5855 50  0000 L CNN
 F 2 "Package_TO_SOT_THT:TO-220-3_Vertical" H 8550 5825 50  0001 L CIN
@@
 $EndComp
 $Comp
-L Regulator_Linear:LD1117S33TR_SOT223 U?
+L Regulator_Linear:LD1117S33TR_SOT223 U1
 U 1 1 5FAD8FE3
 P 2400 2950
-F 0 "U?" H 2400 3192 50  0000 C CNN
+F 0 "U1" H 2400 3192 50  0000 C CNN
 F 1 "LD1117V33TR" H 2400 3101 50  0000 C CNN
 F 2 "Package_TO_SOT_SMD:SOT-223-3_TabPin2" H 2400 3150 50  0001 C CNN
@@
 $EndComp
 $Comp
-L Connector:Conn_01x03_Male J?
+L Connector:Conn_01x03_Male J1
 U 1 1 5FADBC04
 P 1250 3050
-F 0 "J?" H 1358 3331 50  0000 C CNN
+F 0 "J1" H 1358 3331 50  0000 C CNN
 F 1 "GX12 male 3p" H 1350 2850 50  0000 C CNN
 F 2 "" H 1250 3050 50  0001 C CNN
@@
 $EndComp
 $Comp
-L Device:Antenna AE?
+L Device:Antenna AE1
 U 1 1 5FAE0B60
 P 9550 1100
-F 0 "AE?" H 9630 1089 50  0000 L CNN
+F 0 "AE1" H 9630 1089 50  0000 L CNN
 F 1 "Antenna" H 9630 998 50  0000 L CNN
 F 2 "" H 9550 1100 50  0001 C CNN
@@
 $EndComp
 $Comp
-L Device:R R?
+L Device:R R3
 U 1 1 5FAE1AAF
 P 7600 5900
-F 0 "R?" V 7393 5900 50  0000 C CNN
+F 0 "R3" V 7393 5900 50  0000 C CNN
 F 1 "2k2" V 7484 5900 50  0000 C CNN
 F 2 "" V 7530 5900 50  0001 C CNN
@@
 $EndComp
 $Comp
-L Connector:Conn_01x04_Male J?
+L Connector:Conn_01x04_Male J4
 U 1 1 5FAE59B2
 P 9900 3400
-F 0 "J?" H 9872 3374 50  0000 R CNN
+F 0 "J4" H 9872 3374 50  0000 R CNN
 F 1 "GX12 Male 4p" H 10200 3100 50  0000 R CNN
 F 2 "" H 9900 3400 50  0001 C CNN
@@
 $EndComp
 $Comp
-L Connector:Conn_01x02_Male J?
+L Connector:Conn_01x02_Male J5
 U 1 1 5FAEBB54
 P 9900 4450
-F 0 "J?" H 9872 4424 50  0000 R CNN
+F 0 "J5" H 9872 4424 50  0000 R CNN
 F 1 "GX12 Male 2p" H 10200 4250 50  0000 R CNN
 F 2 "" H 9900 4450 50  0001 C CNN
@@
 $EndComp
 $Comp
-L Connector:Conn_01x05_Male J?
+L Connector:Conn_01x05_Male J6
 U 1 1 5FAECD87
 P 9900 5750
-F 0 "J?" H 9872 5774 50  0000 R CNN
+F 0 "J6" H 9872 5774 50  0000 R CNN
 F 1 "GX12 Male 5p" H 10200 5450 50  0000 R CNN
 F 2 "" H 9900 5750 50  0001 C CNN
@@
 $EndComp
 $Comp
-L RF_Module:RFM69HW U?
+L RF_Module:RFM69HW U2
 U 1 1 5FAD1D3E
 P 7850 2350
-F 0 "U?" V 7896 1806 50  0000 R CNN
+F 0 "U2" V 7896 1806 50  0000 R CNN
 F 1 "RFM69HW" V 8050 1750 50  0000 R CNN
 F 2 "RF_Module:HOPERF_RFM69HW" H 7850 1750 50  0001 C CNN
@@
 Wind
 $Comp
-L power:+3.3V #PWR?
+L power:+3.3V #PWR05
 U 1 1 5FB1C424
 P 3400 2800
-F 0 "#PWR?" H 3400 2650 50  0001 C CNN
+F 0 "#PWR05" H 3400 2650 50  0001 C CNN
 F 1 "+3.3V" H 3415 2973 50  0000 C CNN
 F 2 "" H 3400 2800 50  0001 C CNN
@@
 $EndComp
 $Comp
-L power:GND #PWR?
+L power:GND #PWR04
 U 1 1 5FB1CEF5
 P 2400 3550
-F 0 "#PWR?" H 2400 3300 50  0001 C CNN
+F 0 "#PWR04" H 2400 3300 50  0001 C CNN
 F 1 "GND" H 2405 3377 50  0000 C CNN
 F 2 "" H 2400 3550 50  0001 C CNN
@@
 	3400 2800 3400 2950
 $Comp
-L power:+3.3V #PWR?
+L power:+3.3V #PWR014
 U 1 1 5FB1F1D8
 P 9350 3200
-F 0 "#PWR?" H 9350 3050 50  0001 C CNN
+F 0 "#PWR014" H 9350 3050 50  0001 C CNN
 F 1 "+3.3V" H 9365 3373 50  0000 C CNN
 F 2 "" H 9350 3200 50  0001 C CNN
@@
 $EndComp
 $Comp
-L power:+3.3V #PWR?
+L power:+3.3V #PWR017
 U 1 1 5FB206F9
 P 9350 5400
-F 0 "#PWR?" H 9350 5250 50  0001 C CNN
+F 0 "#PWR017" H 9350 5250 50  0001 C CNN
 F 1 "+3.3V" H 9365 5573 50  0000 C CNN
 F 2 "" H 9350 5400 50  0001 C CNN
@@
 $EndComp
 $Comp
-L power:+3.3V #PWR?
+L power:+3.3V #PWR013
 U 1 1 5FB217D5
 P 8950 3950
-F 0 "#PWR?" H 8950 3800 50  0001 C CNN
+F 0 "#PWR013" H 8950 3800 50  0001 C CNN
 F 1 "+3.3V" H 8965 4123 50  0000 C CNN
 F 2 "" H 8950 3950 50  0001 C CNN
@@
 $EndComp
 $Comp
-L power:GND #PWR?
+L power:GND #PWR015
 U 1 1 5FB21DAF
 P 9350 3650
-F 0 "#PWR?" H 9350 3400 50  0001 C CNN
+F 0 "#PWR015" H 9350 3400 50  0001 C CNN
 F 1 "GND" H 9355 3477 50  0000 C CNN
 F 2 "" H 9350 3650 50  0001 C CNN
@@
 $EndComp
 $Comp
-L power:GND #PWR?
+L power:GND #PWR016
 U 1 1 5FB22F76
 P 9350 4600
-F 0 "#PWR?" H 9350 4350 50  0001 C CNN
+F 0 "#PWR016" H 9350 4350 50  0001 C CNN
 F 1 "GND" H 9355 4427 50  0000 C CNN
 F 2 "" H 9350 4600 50  0001 C CNN
@@
 $EndComp
 $Comp
-L power:GND #PWR?
+L power:GND #PWR018
 U 1 1 5FB2F00C
 P 9350 6050
-F 0 "#PWR?" H 9350 5800 50  0001 C CNN
+F 0 "#PWR018" H 9350 5800 50  0001 C CNN
 F 1 "GND" H 9355 5877 50  0000 C CNN
 F 2 "" H 9350 6050 50  0001 C CNN
@@
 $EndComp
 $Comp
-L power:+12V #PWR?
+L power:+12V #PWR01
 U 1 1 5FB34165
 P 1800 2800
-F 0 "#PWR?" H 1800 2650 50  0001 C CNN
+F 0 "#PWR01" H 1800 2650 50  0001 C CNN
 F 1 "+12V" H 1815 2973 50  0000 C CNN
 F 2 "" H 1800 2800 50  0001 C CNN
@@
 	1800 2950 2100 2950
 $Comp
-L power:+12V #PWR?
+L power:+12V #PWR09
 U 1 1 5FB34E10
-P 8450 5400
-F 0 "#PWR?" H 8450 5250 50  0001 C CNN
-F 1 "+12V" H 8465 5573 50  0000 C CNN
-F 2 "" H 8450 5400 50  0001 C CNN
-F 3 "" H 8450 5400 50  0001 C CNN
-	1    8450 5400
-	1    0    0    -1
-$EndComp
-$Comp
-L power:GND #PWR?
+P 8450 5100
+F 0 "#PWR09" H 8450 4950 50  0001 C CNN
+F 1 "+12V" H 8465 5273 50  0000 C CNN
+F 2 "" H 8450 5100 50  0001 C CNN
+F 3 "" H 8450 5100 50  0001 C CNN
+	1    8450 5100
+	1    0    0    -1
+$EndComp
+$Comp
+L power:GND #PWR010
 U 1 1 5FB37CB4
 P 8450 6150
-F 0 "#PWR?" H 8450 5900 50  0001 C CNN
+F 0 "#PWR010" H 8450 5900 50  0001 C CNN
 F 1 "GND" H 8455 5977 50  0000 C CNN
 F 2 "" H 8450 6150 50  0001 C CNN
@@
 	8450 6150 8450 6100
 Wire Wire Line
-	8450 5400 8450 5550
-Wire Wire Line
-	8450 5550 9700 5550
-Wire Wire Line
 	9700 5650 8450 5650
 Wire Wire Line
@@
 	7650 1850 7650 1350
 $Comp
-L power:+3.3V #PWR?
+L power:+3.3V #PWR07
 U 1 1 5FB3D738
 P 7000 2200
-F 0 "#PWR?" H 7000 2050 50  0001 C CNN
+F 0 "#PWR07" H 7000 2050 50  0001 C CNN
 F 1 "+3.3V" H 7015 2373 50  0000 C CNN
 F 2 "" H 7000 2200 50  0001 C CNN
@@
 	7000 2350 7000 2200
 $Comp
-L power:GND #PWR?
+L power:GND #PWR011
 U 1 1 5FB3E6DB
 P 8500 2550
-F 0 "#PWR?" H 8500 2300 50  0001 C CNN
+F 0 "#PWR011" H 8500 2300 50  0001 C CNN
 F 1 "GND" H 8505 2377 50  0000 C CNN
 F 2 "" H 8500 2550 50  0001 C CNN
@@
 	8500 2250 8500 2550
 $Comp
-L Device:CP1 C?
+L Device:CP1 47uF1
 U 1 1 5FB4097F
 P 7000 2650
-F 0 "C?" H 7115 2696 50  0000 L CNN
+F 0 "47uF1" H 6600 2650 50  0000 L CNN
 F 1 "CP1" H 7115 2605 50  0000 L CNN
 F 2 "" H 7000 2650 50  0001 C CNN
@@
 	6650 1350 7650 1350
 $Comp
-L power:GND #PWR?
+L power:GND #PWR08
 U 1 1 5FB596B3
 P 7000 2950
-F 0 "#PWR?" H 7000 2700 50  0001 C CNN
+F 0 "#PWR08" H 7000 2700 50  0001 C CNN
 F 1 "GND" H 7005 2777 50  0000 C CNN
 F 2 "" H 7000 2950 50  0001 C CNN
@@
 	5600 3850 7100 3850
 $Comp
-L Device:R R?
+L Device:R R2
 U 1 1 5FB6D848
 P 6700 6150
-F 0 "R?" H 6630 6196 50  0000 R CNN
+F 0 "R2" H 6630 6196 50  0000 R CNN
 F 1 "2k2" H 6630 6105 50  0000 R CNN
 F 2 "" V 6630 6150 50  0001 C CNN
@@
 $EndComp
 $Comp
-L power:+3.3V #PWR?
+L power:+3.3V #PWR06
 U 1 1 5FB6DED0
 P 6700 5900
-F 0 "#PWR?" H 6700 5750 50  0001 C CNN
+F 0 "#PWR06" H 6700 5750 50  0001 C CNN
 F 1 "+3.3V" H 6715 6073 50  0000 C CNN
 F 2 "" H 6700 5900 50  0001 C CNN
@@
 	6700 6450 6450 6450
 $Comp
-L Device:R R?
+L Device:R R5
 U 1 1 5FB706FD
 P 8950 4200
-F 0 "R?" H 8880 4246 50  0000 R CNN
+F 0 "R5" H 8880 4246 50  0000 R CNN
 F 1 "4k7" H 8880 4155 50  0000 R CNN
 F 2 "" V 8880 4200 50  0001 C CNN
@@
 	8450 3950 5600 3950
 $Comp
-L Device:R R?
+L Device:R R4
 U 1 1 5FB7DDC3
 P 8800 3150
-F 0 "R?" H 8730 3196 50  0000 R CNN
+F 0 "R4" H 8730 3196 50  0000 R CNN
 F 1 "4k7" H 8730 3105 50  0000 R CNN
 F 2 "" V 8730 3150 50  0001 C CNN
@@
 $EndComp
 $Comp
-L power:+3.3V #PWR?
+L power:+3.3V #PWR012
 U 1 1 5FB7E2C9
 P 8800 2900
-F 0 "#PWR?" H 8800 2750 50  0001 C CNN
+F 0 "#PWR012" H 8800 2750 50  0001 C CNN
 F 1 "+3.3V" H 8815 3073 50  0000 C CNN
 F 2 "" H 8800 2900 50  0001 C CNN
@@
 	9550 1750 9550 1300
 $Comp
-L Device:R R?
+L Device:R R1
 U 1 1 5FB87769
 P 3050 6450
-F 0 "R?" V 3257 6450 50  0000 C CNN
+F 0 "R1" V 3257 6450 50  0000 C CNN
 F 1 "470" V 3166 6450 50  0000 C CNN
 F 2 "" V 2980 6450 50  0001 C CNN
@@
 $EndComp
 $Comp
-L Connector:Conn_01x02_Male J?
+L Connector:Conn_01x02_Male J2
 U 1 1 5FB89C3A
 P 1350 6450
-F 0 "J?" H 1322 6424 50  0000 R CNN
+F 0 "J2" H 1322 6424 50  0000 R CNN
 F 1 "Button LED" H 1650 6250 50  0000 R CNN
 F 2 "" H 1350 6450 50  0001 C CNN
@@
 $EndComp
 $Comp
-L Connector:Conn_01x02_Male J?
+L Connector:Conn_01x02_Male J3
 U 1 1 5FB8B347
 P 1350 7050
-F 0 "J?" H 1322 7024 50  0000 R CNN
+F 0 "J3" H 1322 7024 50  0000 R CNN
 F 1 "Button" H 1650 6850 50  0000 R CNN
 F 2 "" H 1350 7050 50  0001 C CNN
@@
 	2900 6450 1550 6450
 $Comp
-L power:GND #PWR?
+L power:GND #PWR02
 U 1 1 5FB945DD
 P 2050 6550
-F 0 "#PWR?" H 2050 6300 50  0001 C CNN
+F 0 "#PWR02" H 2050 6300 50  0001 C CNN
 F 1 "GND" H 2055 6377 50  0000 C CNN
 F 2 "" H 2050 6550 50  0001 C CNN
@@
 	1550 6550 2050 6550
 $Comp
-L power:GND #PWR?
+L power:GND #PWR03
 U 1 1 5FB96D6D
 P 2050 7150
-F 0 "#PWR?" H 2050 6900 50  0001 C CNN
+F 0 "#PWR03" H 2050 6900 50  0001 C CNN
 F 1 "GND" H 2055 6977 50  0000 C CNN
 F 2 "" H 2050 7150 50  0001 C CNN
@@
 Wire Wire Line
 	2450 7050 1550 7050
+$Comp
+L Device:D D1
+U 1 1 5FBA3DF1
+P 8450 5400
+F 0 "D1" V 8404 5480 50  0000 L CNN
+F 1 "D" V 8495 5480 50  0000 L CNN
+F 2 "" H 8450 5400 50  0001 C CNN
+F 3 "~" H 8450 5400 50  0001 C CNN
+	1    8450 5400
+	0    1    1    0
+$EndComp
+Wire Wire Line
+	8450 5550 8450 5650
+Connection ~ 8450 5650
+Wire Wire Line
+	9700 5550 8900 5550
+Wire Wire Line
+	8900 5550 8900 5150
+Wire Wire Line
+	8900 5150 8450 5150
+Wire Wire Line
+	8450 5150 8450 5100
+Wire Wire Line
+	8450 5250 8450 5150
+Connection ~ 8450 5150
 $EndSCHEMATC
