File: ws3.0/KiCad/ws_3.0/power.kicad_sch (KiCad schematic)
At the start: 9 parts, among them J5 2604-1102, U2 LF33_TO220

Commit message: first ws3.0 draft
Parts:
- R1: value 330 -> 1k
Changed lines of the file:
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@@
+	)
+	(junction
+		(at 50.8 90.17)
+		(diameter 0)
+		(color 0 0 0 0)
 	)
 	(junction
@@
 	)
 	(junction
-		(at 50.8 90.17)
-		(diameter 0)
-		(color 0 0 0 0)
-	)
-	(junction
 		(at 100.33 115.57)
 		(diameter 0)
@@
 		(color 0 0 0 0)
 	)
-	(junction
-		(at 67.31 90.17)
-		(diameter 0)
-		(color 0 0 0 0)
-	)
 	(wire
 		(pts
@@
 	(wire
 		(pts
-			(xy 45.72 90.17) (xy 50.8 90.17)
-		)
-		(stroke
-			(width 0)
-			(type default)
-		)
-	)
-	(wire
-		(pts
 			(xy 76.2 100.33) (xy 93.98 100.33)
 		)
@@
 	(wire
 		(pts
-			(xy 67.31 88.9) (xy 67.31 90.17)
+			(xy 50.8 90.17) (xy 50.8 100.33)
 		)
 		(stroke
@@
 	(wire
 		(pts
+			(xy 50.8 90.17) (xy 93.98 90.17)
+		)
+		(stroke
+			(width 0)
+			(type default)
+		)
+	)
+	(wire
+		(pts
 			(xy 50.8 115.57) (xy 93.98 115.57)
 		)
@@
 	(wire
 		(pts
-			(xy 50.8 100.33) (xy 50.8 90.17)
+			(xy 44.45 90.17) (xy 50.8 90.17)
 		)
 		(stroke
@@
 	(wire
 		(pts
-			(xy 67.31 90.17) (xy 93.98 90.17)
-		)
-		(stroke
-			(width 0)
-			(type default)
-		)
-	)
-	(wire
-		(pts
 			(xy 176.53 115.57) (xy 154.94 115.57)
 		)
@@
 	(wire
 		(pts
+			(xy 50.8 82.55) (xy 50.8 90.17)
+		)
+		(stroke
+			(width 0)
+			(type default)
+		)
+	)
+	(wire
+		(pts
 			(xy 176.53 90.17) (xy 176.53 92.71)
 		)
@@
 		)
 	)
-	(wire
-		(pts
-			(xy 50.8 90.17) (xy 67.31 90.17)
-		)
-		(stroke
-			(width 0)
-			(type default)
-		)
-	)
-	(label "RAW"
-		(at 67.31 88.9 0)
+	(global_label "RAW"
+		(shape input)
+		(at 44.45 90.17 180)
+		(fields_autoplaced yes)
 		(effects
 			(font
 				(size 1.27 1.27)
 			)
-			(justify left bottom)
+			(justify right)
+		)
+		(property "Intersheetrefs" "${INTERSHEET_REFS}"
+			(at 37.6548 90.17 0)
+			(effects
+				(font
+					(size 1.27 1.27)
+				)
+				(justify right)
+				(hide yes)
+			)
 		)
 	)
@@
 			)
 		)
-		(property "Value" "330"
+		(property "Value" "1k"
 			(at 179.07 109.2199 0)
 			(effects
@@
 	(symbol
 		(lib_id "power:PWR_FLAG")
-		(at 45.72 90.17 90)
+		(at 50.8 82.55 90)
 		(unit 1)
 		(exclude_from_sim no)
@@
 		(fields_autoplaced yes)
 		(property "Reference" "#FLG02"
-			(at 43.815 90.17 0)
+			(at 48.895 82.55 0)
 			(effects
 				(font
@@
 		)
 		(property "Value" "PWR_FLAG"
-			(at 41.91 90.1699 90)
+			(at 46.99 82.5499 90)
 			(effects
 				(font
@@
 		)
 		(property "Footprint" ""
-			(at 45.72 90.17 0)
+			(at 50.8 82.55 0)
 			(effects
 				(font
@@
 		)
 		(property "Datasheet" "~"
-			(at 45.72 90.17 0)
+			(at 50.8 82.55 0)
 			(effects
 				(font
@@
 		)
 		(property "Description" "Special symbol for telling ERC where power comes from"
-			(at 45.72 90.17 0)
-			(effects
-				(font
+			(at 50.8 82.55 0)
+			(effects
+				(font
