File: ws3.0/KiCad/ws_3.0/radio.kicad_sch (KiCad schematic)
At the start: 11 parts, among them J3 Wind, J4 Temp, SW1 SW_DIP_x03, U5 RFM95W-868S2

Commit message: first ws3.0 draft
Parts:
- removed AE1: Antenna, boan_devices:Antenna 868MHz, symbol Device:Antenna
- removed C8: 1000uF, Capacitor_THT:CP_Radial_D10.0mm_P5.00mm, symbol Device:C_Polarized
- removed R5, R6, R7: 4k7, Resistor_SMD:R_0805_2012Metric_Pad1.20x1.40mm_HandSolder, symbol Device:R
- removed SW1: SW_DIP_x03, Button_Switch_THT:SW_DIP_SPSTx03_Slide_9.78x9.8mm_W7.62mm_P2.54mm, symbol Switch:SW_DIP_x03
- removed U5: RFM95W-868S2, boan_devices:HOPERF_RFM9XW_SMD, symbol RF_Module:RFM95W-868S2
