File: ws3.0/KiCad/ws_3.0/attiny85.kicad_sch (KiCad schematic)
At the start: 17 parts, among them J1 ISP TINY, J2 Rain, SW2 RESET TINY, U3 ATtiny85V-10S, U4 XC6206PxxxMR

Commit message: Updates for mk #5
Parts:
- removed C6, C7: 0.1uF, Capacitor_SMD:C_0805_2012Metric_Pad1.18x1.45mm_HandSolder, symbol Device:C
- added BT2: CR2032, boan_devices:CR2032 standing 1074, symbol boan_devices:Battery_Cell_3p
- added JP1: SCL, boan_devices:Jumper 2p, symbol boan_devices:Jumper
- added JP2: SDA, boan_devices:Jumper 2p, symbol boan_devices:Jumper
- added JP3: CLEAR, boan_devices:Jumper 2p, symbol boan_devices:Jumper
- added R5: 4k7, Resistor_SMD:R_0805_2012Metric_Pad1.20x1.40mm_HandSolder, symbol Device:R
- D2: value 1N5819WS -> BAP70; footprint boan_devices:1N5819HW -> boan_devices:BAP70
- U4: footprint Package_TO_SOT_SMD:SOT-23-3 -> boan_devices:SOT-23
Connections:
- net +3.3V: no longer D3.2 (A), J1.2 (VCC), R11.2
- net BACKUP_POWER: now also R11.2, R5.1
- net GND: now also BT2.2 (-), JP3.1; no longer BT1.2 (-)
- net I2C_SCL: now also JP1.2; no longer J1.3 (SCK), U3.7 (PB2)
- net I2C_SDA: now also JP2.2; no longer J1.4 (MOSI), U3.5 (AREF/PB0)
- net OPT_CLEAR: now also JP3.2, R5.2
- new net: J1.4 (MOSI), JP2.1, U3.5 (AREF/PB0)
- new net: J1.3 (SCK), JP1.1, U3.7 (PB2)
- new net BAT: BT1.2 (-), BT2.1 (+), BT2.3
- new net RAW: D3.2 (A), J1.2 (VCC)
Other:
- note added: "2 x CR2032 = 2 x 3.3V = 6.6V 6.6V - 0.9-1.1V (BAP70) = 5.6V ok for Vin of max 6V"
- note added: "PROGRAM TINY"
- note added: "Vin = 4.0V-6.0V"
- moved on the sheet: J1, R11, R3, R4

Commit message: PCBWAYs delivery 2025-04-16 mk#5 of ws3.0
Parts:
- removed C3: 0.1uF, Capacitor_SMD:C_0805_2012Metric_Pad1.18x1.45mm_HandSolder, symbol Device:C
- removed JP1: SCL, boan_devices:Jumper 2p, symbol boan_devices:Jumper
- removed JP2: SDA, boan_devices:Jumper 2p, symbol boan_devices:Jumper
- removed JP3: CLEAR, boan_devices:Jumper 2p, symbol boan_devices:Jumper
- removed R5: 4k7, Resistor_SMD:R_0805_2012Metric_Pad1.20x1.40mm_HandSolder, symbol Device:R
- added R6: 4k7, Resistor_SMD:R_0805_2012Metric_Pad1.20x1.40mm_HandSolder, symbol Device:R
- added SW1: SW_DIP_x04, Button_Switch_THT:SW_DIP_SPSTx04_Slide_9.78x12.34mm_W7.62mm_P2.54mm, symbol Switch:SW_DIP_x04
Connections:
- net BACKUP_POWER: now also R6.1
- net GND: now also J2.4, SW1.3, SW1.4
- net I2C_SCL: now also SW1.8
- net I2C_SDA: now also SW1.7
- net OPT_CLEAR: now also R6.2, SW1.6
- net at J1.4 (MOSI), U3.5 (AREF/PB0): now also SW1.2
- net at J1.3 (SCK), U3.7 (PB2): now also SW1.1
- net BATTERY renamed BACKUP_BATTERY
- new net DISABLE_RADIO: SW1.5
Other:
- note added: "Powers the board LDO"
- note removed: "PROGRAM TINY"
- moved on the sheet: R3, R4
