File: ws3.0/KiCad/ws_3.0/ws_3.0.kicad_sch (KiCad schematic)
At the start: 14 parts, among them J6 ISP MEGA, J7 FTDI MEGA, SW3 RESET ATMEGA, U1 ATmega328P-A, Y1 Crystal

Commit message: Updates for mk #5
Parts:
- added AE1: Antenna, boan_devices:Antenna 868MHz, symbol Device:Antenna
- added C1: 0.1uF, Capacitor_SMD:C_0805_2012Metric_Pad1.18x1.45mm_HandSolder, symbol Device:C
- added C2: 2.2uF, Capacitor_THT:CP_Radial_D5.0mm_P2.00mm, symbol Device:C_Polarized
- added C8: 1000uF, Capacitor_THT:CP_Radial_D10.0mm_P5.00mm, symbol Device:C_Polarized
- added D1: GREEN, LED_SMD:LED_0805_2012Metric_Pad1.15x1.40mm_HandSolder, symbol Device:LED
- added J3: Wind, boan_devices:RJ10 Horizontal, symbol Connector:RJ10
- added J4: Temp, boan_devices:RJ10 Horizontal, symbol Connector:RJ10
- added J5: 2604-1102, boan_devices:wago 26041102, symbol wago:2604-1102
- added JP4: PROGRAM MEGA, boan_devices:Jumper 2p, symbol boan_devices:Jumper
- added JP5: DEBUG, boan_devices:Jumper 2p, symbol boan_devices:Jumper
- added R1: 1k, Resistor_SMD:R_0805_2012Metric_Pad1.20x1.40mm_HandSolder, symbol Device:R
- added R13, R9: 4k7, Resistor_SMD:R_0805_2012Metric_Pad1.20x1.40mm_HandSolder, symbol Device:R
- added R8: 2k2, Resistor_SMD:R_0805_2012Metric_Pad1.20x1.40mm_HandSolder, symbol Device:R
- added TP1: 12V, Connector_Pin:Pin_D1.0mm_L10.0mm, symbol Connector:TestPoint_Probe
- added TP2: 3.3V, Connector_Pin:Pin_D1.0mm_L10.0mm, symbol Connector:TestPoint_Probe
- added TP3: GND, Connector_Pin:Pin_D1.0mm_L10.0mm, symbol Connector:TestPoint_Probe
- added U2: LF33_TO220, Package_TO_SOT_THT:TO-220-3_Vertical, symbol Regulator_Linear:LF33_TO220
- added U5: RFM95W-868S2, boan_devices:HOPERF_RFM9XW_SMD, symbol RF_Module:RFM95W-868S2
Connections:
- net +3.3V: now also C2.1, C8.1, D1.2 (A), J3.1, J4.3, R13.1, R8.1, R9.1, TP2.1, U2.3 (VO), U5.13 (3.3V); no longer J6.2 (VCC)
- net DIO0: now also U5.14 (DIO0)
- net GND: now also C1.2, C2.2, C8.2, J3.3, J4.4, J5.3 (2.1), J5.4 (2.2), JP4.1, JP5.1, R1.2, TP3.1, U2.2 (GND), U5.1 (GND), U5.10 (GND), U5.8 (GND)
- net MISO: now also U5.2 (MISO)
- net MOSI: now also U5.3 (MOSI)
- net OPT_DEBUG: now also JP5.2, R13.2
- net SCK: now also U5.4 (SCK)
- net TEMP_1W: now also J4.1, R8.2
- net WIND_DIR: now also J3.2
- net WIND_SPEED: now also J3.4, R9.2
- net at C12.1, R12.1, SW3.1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: now also J6.5 (~{RST})
- net SS renamed NSS
- net NSS: now also U5.5 (NSS); no longer J6.5 (~{RST})
- new net: D1.1 (K), R1.1
- new net: JP4.2, U5.6 (RESET)
- new net ANTENNA: AE1.1 (A), U5.9 (ANT)
- new net RAW: C1.1, J5.1 (1.1), J5.2 (1.2), J6.2 (VCC), TP1.1, U2.1 (VI)
Other:
- removed sheet power
- removed sheet radio and sensors
- note added: "Vin=2.5-16V"
- moved on the sheet: C10, C11, C12, C13, C14, C9, D4, J6, J7, R10, R12, SW3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

Commit message: PCBWAYs delivery 2025-04-16 mk#5 of ws3.0
Parts:
- removed C9: 0.1uF, Capacitor_SMD:C_0805_2012Metric_Pad1.18x1.45mm_HandSolder, symbol Device:C
- removed JP4: PROGRAM MEGA, boan_devices:Jumper 2p, symbol boan_devices:Jumper
- removed JP5: DEBUG, boan_devices:Jumper 2p, symbol boan_devices:Jumper
- added C15, C16: 0.1uF, Capacitor_SMD:C_0805_2012Metric_Pad1.18x1.45mm_HandSolder, symbol Device:C
- added Q1: ISS55EP06LMXTSA1, Package_TO_SOT_SMD:SOT-23_Handsoldering, symbol boan_devices:MOSFET_P-CH_ISS55EP06LMXTSA1
- added R14: 100k, Resistor_SMD:R_0805_2012Metric_Pad1.20x1.40mm_HandSolder, symbol Device:R
- added R15, R16: 560k, Resistor_SMD:R_0805_2012Metric_Pad1.20x1.40mm_HandSolder, symbol Device:R
- R13: value 4k7 -> 100k
Connections:
- net +3.3V: no longer R13.1
- net GND: now also R13.1, C15.2, C16.2, R14.1
- net RAW: now also R16.2
- net at U1.19 (ADC6): now also C15.1, R14.2, R16.1
- net at U1.22 (ADC7): now also R13.2, C16.1, R15.1
- net BACKUP_DIV_CTRL: now reaches U1.26 (PC3)
- net BACKUP_DIV_CTRL: now also Q1.1
- net DISABLE_RADIO: now reaches U5.6 (RESET)
- net OPT_DEBUG: no longer names the net of U1.9 (PD5)
- net OPT_DEBUG: no longer R13.2
- new net: Q1.3, R15.2
- new net BACKUP_BATTERY: Q1.2
Other:
- note added: "Dynamic control of measurment of backup battery or voltage divider will drain them"
- note added: "Leave AREF floating Code uses: DEFAULT (internal up to VCC) INTERNAL (for 1.1V measure)"
- note added: "Powers the board LDO"
- moved on the sheet: C10, C11, C12, C13, C14, D4, J6, J7, R10, R12, SW3, U1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
